Commit message: fixed inverse kinematics for arm. now the arm can enter target position for the arm

File: robot_arm/urdf/model.urdf (robot description, URDF)
Before this commit: robot arm, 11 links, 10 joints
Joints:
- joint connector2_to_link6: limit lower=-1.57 upper=1.57 effort=10 velocity=1 -> lower=-3.14 upper=3.14 effort=10 velocity=1
- joint link1_to_link2: limit lower=-1.57 upper=1.57 effort=10 velocity=1 -> lower=-3.14 upper=3.14 effort=10 velocity=1
- joint link2_to_link3: limit lower=-1.57 upper=1.57 effort=10 velocity=1 -> lower=-3.14 upper=3.14 effort=10 velocity=1; origin xyz=0 0 0.5 -> xyz=0.5 0 0
- joint link3_to_link4: origin xyz=0 0 0.5 -> xyz=0.5 0 0
- joint link4_to_link5: limit lower=-1.57 upper=1.57 effort=10 velocity=1 -> lower=-3.14 upper=3.14 effort=10 velocity=1

Commit message: changed the wrist rotations to be on the XYZ axis to reduce ambiguity. The last link now points downwards (in the -Z direction)

File: robot_arm/urdf/model.urdf (robot description, URDF)
Before this commit: robot arm, 9 links, 8 joints
Joints:
- joint link4_to_link5_roll: axis 1 0 0 -> 0 0 1
- joint link5_to_end: origin xyz=${l5_len} 0 0 rpy=0 0 0 -> xyz=0 0 -${l5_len} rpy=0 0 0
